Commit message: Module 2 changed

File: module_2_simulation/assets/humanoid.urdf (robot description, URDF)
Before this commit: robot simple_humanoid, 11 links, 10 joints
Links:
- removed link base_link
- added link base, mass 1e-3
- added link left_foot, mass 2; collision box size=0.2 0.09 0.14; visual box size=0.2 0.09 0.14
- added link left_hand, mass 0.8; collision capsule length=0.1 radius=0.035; visual capsule length=0.1 radius=0.035
- added link left_toe, mass 0.5; collision box size=0.16 0.07 0.05; visual box size=0.16 0.07 0.05
- added link pelvis, mass 8; collision box size=0.35 0.2 0.1; visual box size=0.35 0.2 0.1
- added link right_foot, mass 2; collision box size=0.2 0.09 0.14; visual box size=0.2 0.09 0.14
- added link right_hand, mass 0.8; collision capsule length=0.1 radius=0.035; visual capsule length=0.1 radius=0.035
- added link right_toe, mass 0.5; collision box size=0.16 0.07 0.05; visual box size=0.16 0.07 0.05
- link head: mass None -> 4; geometry collision sphere radius=0.12; visual sphere radius=0.12
- link left_lower_arm: mass None -> 1.8; geometry collision capsule length=0.25 radius=0.04; visual capsule length=0.25 radius=0.04
- link left_shin: mass None -> 4.5; geometry collision capsule length=0.4 radius=0.07; visual capsule length=0.4 radius=0.07
- link left_thigh: mass None -> 6; geometry collision capsule length=0.4 radius=0.08; visual capsule length=0.4 radius=0.08
- link left_upper_arm: mass None -> 2.5; geometry collision capsule length=0.3 radius=0.05; visual capsule length=0.3 radius=0.05
- link right_lower_arm: mass None -> 1.8; geometry collision capsule length=0.25 radius=0.04; visual capsule length=0.25 radius=0.04
- link right_shin: mass None -> 4.5; geometry collision capsule length=0.4 radius=0.07; visual capsule length=0.4 radius=0.07
- link right_thigh: mass None -> 6; geometry collision capsule length=0.4 radius=0.08; visual capsule length=0.4 radius=0.08
- link right_upper_arm: mass None -> 2.5; geometry collision capsule length=0.3 radius=0.05; visual capsule length=0.3 radius=0.05
- link torso: mass 10 -> 12; geometry collision box size=0.3 0.22 0.5; visual box size=0.3 0.22 0.5
Joints:
- removed joint base_to_torso
- added joint base_to_pelvis: type fixed, parent base, child pelvis, origin xyz=0 0 1.0
- added joint left_ankle: type fixed, parent left_shin, child left_foot, origin xyz=0 0 -0.4
- added joint left_toe: type fixed, parent left_foot, child left_toe, origin xyz=0.1 0 -0.05
- added joint left_wrist: type fixed, parent left_lower_arm, child left_hand, origin xyz=0 0 -0.25
- added joint right_ankle: type fixed, parent right_shin, child right_foot, origin xyz=0 0 -0.4
- added joint right_toe: type fixed, parent right_foot, child right_toe, origin xyz=0.1 0 -0.05
- added joint right_wrist: type fixed, parent right_lower_arm, child right_hand, origin xyz=0 0 -0.25
- added joint spine: type fixed, parent pelvis, child torso, origin xyz=0 0 0.1
- joint left_elbow: axis 0 1 0 -> 1 0 0; limit lower=0 upper=1.5 effort=10 velocity=1.0 -> lower=-1.0 upper=1.5 effort=80 velocity=3.0
- joint left_hip: limit lower=-1.0 upper=1.0 effort=20 velocity=1.0 -> lower=-1.2 upper=1.2 effort=200 velocity=3.0; origin xyz=0.1 0 0 -> xyz=0 0.09 0; parent torso -> pelvis
- joint left_knee: limit lower=0 upper=1.5 effort=20 velocity=1.0 -> lower=0 upper=1.7 effort=180 velocity=3.0
- joint left_shoulder: axis 0 1 0 -> 1 0 0; limit lower=-1.5 upper=1.5 effort=15 velocity=1.0 -> lower=-1.5 upper=1.5 effort=120 velocity=3.0; origin xyz=0.25 0 0.45 -> xyz=0 0.17 0.45
- joint neck: axis 0 1 0 -> (none); limit lower=-1.0 upper=1.0 effort=5 velocity=1.0 -> (none); origin xyz=0 0 0.6 -> xyz=0 0 0.5; type revolute -> fixed
- joint right_elbow: axis 0 1 0 -> 1 0 0; limit lower=0 upper=1.5 effort=10 velocity=1.0 -> lower=-1.0 upper=1.5 effort=80 velocity=3.0
- joint right_hip: limit lower=-1.0 upper=1.0 effort=20 velocity=1.0 -> lower=-1.2 upper=1.2 effort=200 velocity=3.0; origin xyz=-0.1 0 0 -> xyz=0 -0.09 0; parent torso -> pelvis
- joint right_knee: limit lower=0 upper=1.5 effort=20 velocity=1.0 -> lower=0 upper=1.7 effort=180 velocity=3.0
- joint right_shoulder: axis 0 1 0 -> 1 0 0; limit lower=-1.5 upper=1.5 effort=15 velocity=1.0 -> lower=-1.5 upper=1.5 effort=120 velocity=3.0; origin xyz=-0.25 0 0.45 -> xyz=0 -0.17 0.45
